File: BeeBeeAte-RemoteBoard.sch (EAGLE design)
At the start: 56 parts, among them IC1 CP2102, J1 3-1734035-2, T1 S8050, T2 S8050, U1 ESP32-WROOM-32, U2 LM5.0

Commit message: Added 3D Files and modified Board
Parts:
- removed D3: 1N4007, Diodes:1N4007
- added R18: 0, rcl:R-EU_R0805
Connections:
- net 5V: now also R18.2; no longer D3.A
- net VBUS: now also R18.1; no longer D3.C
