File: BeeBeeAte-BotBoard.sch (EAGLE design)
At the start: 100 parts, among them IC1 CP2102, J1 3-1734035-2, T1 S8050, T2 S8050, U1 ESP32-WROOM-32, U2 LM5.0, U3 DRIVER 2, U4 DRIVER 1, U5 DRIVER 3, U6 DRIVER 4

Commit message: Added 3,7V battery
Parts:
- added U$28: 9V+, 03lanfra-PADS:LITZENPAD
- added U$29: 9V-, 03lanfra-PADS:LITZENPAD
- added U$30: 9VSW+, 03lanfra-PADS:LITZENPAD
- added U$31: 9VSW-, 03lanfra-PADS:LITZENPAD
Connections:
- new net 9V: R11.1, R5.1, U$31.P$1
- new net N$15: U$28.P$1, U$30.P$1
- net GND: now also U$29.P$1
- net VCC: no longer R11.1, R5.1
Other:
- note added: "D3 weglassen"
- note added: "Eventuell 0Ohm"
- moved on the sheet: R5
Changed lines of the file:
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@@
 <part name="FRAME1" library="frames" library_urn="urn:adsk.eagle:library:229" deviceset="A4L-LOC" device="" value="Power Supply"/>
 <part name="FRAME4" library="frames" library_urn="urn:adsk.eagle:library:229" deviceset="A4L-LOC" device="" value="MPU6050"/>
+<part name="U$28" library="03lanfra-PADS" deviceset="LITZENPAD" device="" value="9V+"/>
+<part name="U$29" library="03lanfra-PADS" deviceset="LITZENPAD" device="" value="9V-"/>
+<part name="U$30" library="03lanfra-PADS" deviceset="LITZENPAD" device="" value="9VSW+"/>
+<part name="U$31" library="03lanfra-PADS" deviceset="LITZENPAD" device="" value="9VSW-"/>
 </parts>
 <sheets>
@@
 <attribute name="VALUE" x="127" y="96.52" size="1.778" layer="96"/>
 </instance>
-<instance part="R5" gate="G$1" x="121.92" y="114.3" smashed="yes">
-<attribute name="NAME" x="118.11" y="115.7986" size="1.778" layer="95"/>
-<attribute name="VALUE" x="118.11" y="110.998" size="1.778" layer="96"/>
+<instance part="R5" gate="G$1" x="114.3" y="114.3" smashed="yes">
+<attribute name="NAME" x="110.49" y="115.7986" size="1.778" layer="95"/>
+<attribute name="VALUE" x="110.49" y="110.998" size="1.778" layer="96"/>
 </instance>
 <instance part="D1" gate="G$1" x="154.94" y="121.92" smashed="yes" rot="R180">
@@
 <attribute name="LAST_DATE_TIME" x="217.17" y="10.16" size="2.286" layer="94"/>
 <attribute name="SHEET" x="230.505" y="5.08" size="2.54" layer="94"/>
+</instance>
+<instance part="U$28" gate="G$1" x="43.18" y="119.38" smashed="yes" rot="R270">
+<attribute name="NAME" x="45.72" y="121.92" size="1.27" layer="95" rot="R270"/>
+<attribute name="VALUE" x="39.37" y="121.92" size="1.27" layer="96" rot="R270"/>
+</instance>
+<instance part="U$29" gate="G$1" x="50.8" y="119.38" smashed="yes" rot="R270">
+<attribute name="NAME" x="53.34" y="121.92" size="1.27" layer="95" rot="R270"/>
+<attribute name="VALUE" x="46.99" y="121.92" size="1.27" layer="96" rot="R270"/>
+</instance>
+<instance part="U$30" gate="G$1" x="43.18" y="106.68" smashed="yes" rot="R90">
+<attribute name="NAME" x="40.64" y="104.14" size="1.27" layer="95" rot="R90"/>
+<attribute name="VALUE" x="46.99" y="104.14" size="1.27" layer="96" rot="R90"/>
+</instance>
+<instance part="U$31" gate="G$1" x="43.18" y="99.06" smashed="yes" rot="R270">
+<attribute name="NAME" x="45.72" y="101.6" size="1.27" layer="95" rot="R270"/>
+<attribute name="VALUE" x="39.37" y="101.6" size="1.27" layer="96" rot="R270"/>
 </instance>
 </instances>
@@
 <label x="73.66" y="83.82" size="1.778" layer="95" rot="R270" xref="yes"/>
 <pinref part="LTZPDGND" gate="G$1" pin="P$1"/>
-</segment>
-<segment>
-<pinref part="R5" gate="G$1" pin="1"/>
-<wire x1="114.3" y1="114.3" x2="116.84" y2="114.3" width="0.1524" layer="91"/>
-<label x="114.3" y="114.3" size="1.778" layer="95" rot="R180" xref="yes"/>
-</segment>
-<segment>
-<pinref part="R11" gate="G$1" pin="1"/>
-<wire x1="114.3" y1="76.2" x2="116.84" y2="76.2" width="0.1524" layer="91"/>
-<label x="114.3" y="76.2" size="1.778" layer="95" rot="R180" xref="yes"/>
 </segment>
 </net>
@@
 <pinref part="GND13" gate="1" pin="GND"/>
 </segment>
+<segment>
+<pinref part="U$29" gate="G$1" pin="P$1"/>
+<wire x1="50.8" y1="114.3" x2="50.8" y2="109.22" width="0.1524" layer="91"/>
+<label x="50.8" y="109.22" size="1.778" layer="95"/>
+</segment>
 </net>
 <net name="N$4" class="0">
 <segment>
-<wire x1="127" y1="114.3" x2="129.54" y2="114.3" width="0.1524" layer="91"/>
+<wire x1="119.38" y1="114.3" x2="129.54" y2="114.3" width="0.1524" layer="91"/>
 <wire x1="129.54" y1="114.3" x2="134.62" y2="114.3" width="0.1524" layer="91"/>
 <pinref part="C2" gate="G$1" pin="1"/>
@@
 </segment>
 </net>
+<net name="N$15" class="0">
+<segment>
+<pinref part="U$28" gate="G$1" pin="P$1"/>
+<pinref part="U$30" gate="G$1" pin="P$1"/>
+<wire x1="43.18" y1="114.3" x2="43.18" y2="111.76" width="0.1524" layer="91"/>
+</segment>
+</net>
+<net name="9V" class="0">
+<segment>
+<pinref part="U$31" gate="G$1" pin="P$1"/>
+<wire x1="43.18" y1="93.98" x2="43.18" y2="88.9" width="0.1524" layer="91"/>
+<label x="43.18" y="88.9" size="1.778" layer="95"/>
+</segment>
+<segment>
+<pinref part="R5" gate="G$1" pin="1"/>
+<wire x1="114.3" y1="114.3" x2="109.22" y2="114.3" width="0.1524" layer="91"/>
+<label x="109.22" y="114.3" size="1.778" layer="95" rot="R180" xref="yes"/>
+</segment>
+<segment>
+<pinref part="R11" gate="G$1" pin="1"/>
+<wire x1="114.3" y1="76.2" x2="116.84" y2="76.2" width="0.1524" layer="91"/>
+<label x="114.3" y="76.2" size="1.778" layer="95" rot="R180" xref="yes"/>
+</segment>
+</net>
 </nets>
 </sheet>
@@
 <plain>
 <text x="22.86" y="127" size="1.778" layer="91">USB</text>
+<text x="147.32" y="119.38" size="1.778" layer="150">D3 weglassen</text>
+<text x="147.32" y="116.84" size="1.778" layer="150">Eventuell 0Ohm</text>
 </plain>
 <instances>

Commit message: Added 3D Files and modified Board
Parts:
- removed D3: 1N4007, Diodes:1N4007
- added R35: 0, rcl:R-EU_R0805
Connections:
- net 5V: now also R35.2; no longer D3.A
- net VBUS: now also R35.1; no longer D3.C
Changed lines of the file:
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@@
 <part name="C7" library="rcl" library_urn="urn:adsk.eagle:library:334" deviceset="C-EU" device="C0805" package3d_urn="urn:adsk.eagle:package:23617/2" value="100n"/>
 <part name="GND10" library="supply1" library_urn="urn:adsk.eagle:library:371" deviceset="GND" device=""/>
-<part name="D3" library="Diodes" library_urn="urn:adsk.eagle:library:11396254" deviceset="1N4007" device="" package3d_urn="urn:adsk.eagle:package:10898391/4"/>
 <part name="R12" library="rcl" library_urn="urn:adsk.eagle:library:334" deviceset="R-EU_" device="R0805" package3d_urn="urn:adsk.eagle:package:23553/2" value="0"/>
 <part name="R13" library="rcl" library_urn="urn:adsk.eagle:library:334" deviceset="R-EU_" device="R0805" package3d_urn="urn:adsk.eagle:package:23553/2" value="0"/>
@@
 <part name="U$30" library="03lanfra-PADS" deviceset="LITZENPAD" device="" value="9VSW+"/>
 <part name="U$31" library="03lanfra-PADS" deviceset="LITZENPAD" device="" value="9VSW-"/>
+<part name="R35" library="rcl" library_urn="urn:adsk.eagle:library:334" deviceset="R-EU_" device="R0805" package3d_urn="urn:adsk.eagle:package:23553/2" value="0"/>
 </parts>
 <sheets>
@@
 <pinref part="U$29" gate="G$1" pin="P$1"/>
 <wire x1="50.8" y1="114.3" x2="50.8" y2="109.22" width="0.1524" layer="91"/>
-<label x="50.8" y="109.22" size="1.778" layer="95"/>
+<label x="50.8" y="109.22" size="1.778" layer="95" rot="R270" xref="yes"/>
 </segment>
 </net>
@@
 <pinref part="U$31" gate="G$1" pin="P$1"/>
 <wire x1="43.18" y1="93.98" x2="43.18" y2="88.9" width="0.1524" layer="91"/>
-<label x="43.18" y="88.9" size="1.778" layer="95"/>
+<label x="43.18" y="88.9" size="1.778" layer="95" rot="R270" xref="yes"/>
 </segment>
 <segment>
@@
 <attribute name="VALUE" x="137.16" y="91.44" size="1.778" layer="96"/>
 </instance>
-<instance part="D3" gate="G$1" x="139.7" y="116.84" smashed="yes" rot="R270">
-<attribute name="NAME" x="142.3416" y="119.1514" size="1.778" layer="95" rot="R270"/>
-<attribute name="VALUE" x="135.2042" y="119.4054" size="1.778" layer="96" rot="R270"/>
-</instance>
 <instance part="R12" gate="G$1" x="154.94" y="96.52" smashed="yes" rot="R90">
 <attribute name="NAME" x="153.4414" y="92.71" size="1.778" layer="95" rot="R90"/>
@@
 <attribute name="NAME" x="204.2414" y="90.17" size="1.778" layer="95" rot="R90"/>
 <attribute name="VALUE" x="209.042" y="90.17" size="1.778" layer="96" rot="R90"/>
+</instance>
+<instance part="R35" gate="G$1" x="139.7" y="119.38" smashed="yes" rot="R90">
+<attribute name="NAME" x="138.2014" y="115.57" size="1.778" layer="95" rot="R90"/>
+<attribute name="VALUE" x="143.002" y="115.57" size="1.778" layer="96" rot="R90"/>
 </instance>
 </instances>
@@
 <net name="5V" class="0">
 <segment>
-<pinref part="D3" gate="G$1" pin="A"/>
-<wire x1="139.7" y1="119.38" x2="139.7" y2="121.92" width="0.1524" layer="91"/>
-<label x="139.7" y="121.92" size="1.778" layer="95" rot="R90" xref="yes"/>
+<label x="139.7" y="129.54" size="1.778" layer="95" rot="R90" xref="yes"/>
+<pinref part="R35" gate="G$1" pin="2"/>
+<wire x1="139.7" y1="129.54" x2="139.7" y2="124.46" width="0.1524" layer="91"/>
 </segment>
 </net>
@@
 <pinref part="C6" gate="G$1" pin="2"/>
 <wire x1="149.86" y1="111.76" x2="149.86" y2="109.22" width="0.1524" layer="91"/>
-<pinref part="D3" gate="G$1" pin="C"/>
 <wire x1="139.7" y1="111.76" x2="139.7" y2="114.3" width="0.1524" layer="91"/>
 <junction x="139.7" y="111.76"/>
@@
 <pinref part="R12" gate="G$1" pin="2"/>
 <wire x1="154.94" y1="111.76" x2="154.94" y2="101.6" width="0.1524" layer="91"/>
-</segment>
-</net>
+<pinref part="R35" gate="G$1" pin="1"/>
+</segment>
+</net>

Commit message: Checked by teacher and fixed
Parts:
- LTZPDGND: value SWITCH - -> SW-
- LTZPDVCC: value SWITCH + -> SW+
Other:
- moved on the sheet: R5
Changed lines of the file:
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@@
 <part name="R11" library="rcl" library_urn="urn:adsk.eagle:library:334" deviceset="R-EU_" device="R0805" package3d_urn="urn:adsk.eagle:package:23553/2" value="0"/>
 <part name="D2" library="Diodes" library_urn="urn:adsk.eagle:library:11396254" deviceset="1N4007" device="" package3d_urn="urn:adsk.eagle:package:10898391/4"/>
-<part name="LTZPDVCC" library="03lanfra-PADS" deviceset="LITZENPAD" device="" value="SWITCH +"/>
-<part name="LTZPDGND" library="03lanfra-PADS" deviceset="LITZENPAD" device="" value="SWITCH -"/>
+<part name="LTZPDVCC" library="03lanfra-PADS" deviceset="LITZENPAD" device="" value="SW+"/>
+<part name="LTZPDGND" library="03lanfra-PADS" deviceset="LITZENPAD" device="" value="SW-"/>
 <part name="U$10" library="03lanfra-PADS" deviceset="MESSPAD" device="" value="GND"/>
 <part name="U$4" library="03lanfra-PADS" deviceset="MESSPAD" device="" value="VCC"/>
@@
 <attribute name="VALUE" x="127" y="96.52" size="1.778" layer="96"/>
 </instance>
-<instance part="R5" gate="G$1" x="114.3" y="114.3" smashed="yes">
-<attribute name="NAME" x="110.49" y="115.7986" size="1.778" layer="95"/>
-<attribute name="VALUE" x="110.49" y="110.998" size="1.778" layer="96"/>
+<instance part="R5" gate="G$1" x="121.92" y="114.3" smashed="yes">
+<attribute name="NAME" x="118.11" y="115.7986" size="1.778" layer="95"/>
+<attribute name="VALUE" x="118.11" y="110.998" size="1.778" layer="96"/>
 </instance>
 <instance part="D1" gate="G$1" x="154.94" y="121.92" smashed="yes" rot="R180">
@@
 <net name="N$4" class="0">
 <segment>
-<wire x1="119.38" y1="114.3" x2="129.54" y2="114.3" width="0.1524" layer="91"/>
+<wire x1="127" y1="114.3" x2="129.54" y2="114.3" width="0.1524" layer="91"/>
 <wire x1="129.54" y1="114.3" x2="134.62" y2="114.3" width="0.1524" layer="91"/>
 <pinref part="C2" gate="G$1" pin="1"/>
@@
 <segment>
 <pinref part="R5" gate="G$1" pin="1"/>
-<wire x1="114.3" y1="114.3" x2="109.22" y2="114.3" width="0.1524" layer="91"/>
-<label x="109.22" y="114.3" size="1.778" layer="95" rot="R180" xref="yes"/>
-</segment>
-<segment>
+<wire x1="114.3" y1="114.3" x2="116.84" y2="114.3" width="0.1524" layer="91"/>
+<label x="114.3" y="114.3" size="1.778" layer="95" rot="R180" xref="yes"/>
+</segment>
+<segment>
