File: EAGLE/BeeBeeAte-RemoteBoard.sch (EAGLE design)
At the start: 56 parts, among them IC1 CP2102, J1 3-1734035-2, T1 S8050, T2 S8050, U1 ESP32-WROOM-32, U2 LM5.0

Commit message: Added Motors
Other:
- note added: "ESP32 und USB-Modul"
- note added: "Joystick"
- note added: "Stromversorgung"
Changed lines of the file:
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@@
 <text x="109.22" y="127" size="1.778" layer="91">3V3 VR</text>
 <text x="109.22" y="93.98" size="1.778" layer="91">5V VR</text>
+<text x="45.72" y="139.7" size="6.4516" layer="97">Stromversorgung</text>
 </plain>
 <instances>
@@
 <plain>
 <text x="66.04" y="121.92" size="1.778" layer="91">USB</text>
+<text x="45.72" y="142.24" size="6.4516" layer="97">ESP32 und USB-Modul</text>
 </plain>
 <instances>
@@
 <description>Joystick</description>
 <plain>
+<text x="86.36" y="119.38" size="6.4516" layer="97">Joystick</text>
 </plain>
 <instances>
