File: EAGLE/Version 2/BeeBeeAte-BotBoardV2.sch (EAGLE design)
At the start: 105 parts, among them IC1 CP2102, J1 3-1734035-2, T1 S8050, T2 S8050, U1 ESP32-WROOM-32, U2 LM5.0, U3 DRIVER 2, U4 DRIVER 1, U5 DRIVER 3, U6 DRIVER 4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

Commit message: New Board
Parts:
- removed LTZPDGND: SW-, 03lanfra-PADS:LITZENPAD
- removed LTZPDVCC: SW+, 03lanfra-PADS:LITZENPAD
- removed R17, R18, R19, R20, R21, R22, R23, R24, R25, R26, R27, R28: 0, rcl:R-EU_R0805
- removed U$1: VCC, 03lanfra-PADS:LITZENPAD
- removed U$10: GND, 03lanfra-PADS:MESSPAD
- removed U$2, U$4: VCC, 03lanfra-PADS:MESSPAD
- removed U$27: GND, 03lanfra-PADS:LITZENPAD
- removed U$28: 9V+, 03lanfra-PADS:LITZENPAD
- removed U$29: 9V-, 03lanfra-PADS:LITZENPAD
- removed U$30: 9VSW+, 03lanfra-PADS:LITZENPAD
- removed U$31: 9VSW-, 03lanfra-PADS:LITZENPAD
- added U$32, U$33, U$34, U$35, U$36: (no value), 03lanfra-PADS:MESSPAD
Connections:
- removed net N$15: U$28.P$1, U$30.P$1
- removed net N$20: R20.2, U3.MS1
- removed net N$21: R21.2, U3.MS2
- removed net N$22: R22.2, U3.MS3
- removed net N$35: R17.2, U5.MS1
- removed net N$36: R18.2, U5.MS2
- removed net N$37: R19.2, U5.MS3
- removed net N$42: R23.2, U4.MS1
- removed net N$43: R24.2, U4.MS2
- removed net N$44: R25.2, U4.MS3
- removed net N$5: LTZPDVCC.P$1, U$1.P$1
- removed net N$53: R26.2, U6.MS1
- removed net N$54: R27.2, U6.MS2
- removed net N$55: R28.2, U6.MS3
- removed net N$57: X1-5.KL
- removed net N$58: X1-6.KL
- removed net N$59: X1-7.KL
- removed net N$60: X1-8.KL
- new net +VCC: U$33.P$1, X1-6.KL, X1-7.KL
- net 3V3: no longer R17.1, R18.1, R19.1, R20.1, R21.1, R22.1, R23.1, R24.1, R25.1, R26.1, R27.1, R28.1
- net 9V: now also U$35.P$1; no longer U$31.P$1
- net GND: now also U$32.P$1, X1-8.KL; no longer U$10.P$1, U$27.P$1, U$29.P$1
- net N$4: no longer U$4.P$1
- net N$46: now also U$36.P$1
- net N$6: now also LED1.C
- net N$8: no longer U$2.P$1
- net N$9: no longer LED1.C
- net VCC: now also U$34.P$1, X1-5.KL; no longer LTZPDGND.P$1
Other:
- note added: "+9V"
- note added: "+VCC"
- note added: "-9V"
- note added: "9V Switch +"
- note added: "9V Switch -"
- note added: "Schalter Out"
- note added: "VCC Switch +"
- note added: "VCC Switch -"
- moved on the sheet: LED1, R10, X1-1, X1-2, X1-3, X1-4, X1-5, X1-6, X1-7, X1-8
