File: EAGLE/Version 2/BeeBeeAte-BotBoardV2.brd (EAGLE design)
At the start: 100 x 100 mm, 105 parts, among them IC1 CP2102, J1 3-1734035-2, T1 S8050, T2 S8050, U1 ESP32-WROOM-32, U2 LM5.0, U3 DRIVER 2, U4 DRIVER 1, U5 DRIVER 3, U6 DRIVER 4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

Commit message: New Board
Parts:
- removed LTZPDGND: SW-, 03lanfra-PADS:LITZENPAD
- removed LTZPDVCC: SW+, 03lanfra-PADS:LITZENPAD
- removed R17, R18, R19, R20, R21, R22, R23, R24, R25, R26, R27, R28: 0, rcl:R0805
- removed U$1: VCC, 03lanfra-PADS:LITZENPAD
- removed U$10: GND, 03lanfra-PADS:MESSPAD
- removed U$2, U$4: VCC, 03lanfra-PADS:MESSPAD
- removed U$27: GND, 03lanfra-PADS:LITZENPAD
- removed U$28: 9V+, 03lanfra-PADS:LITZENPAD
- removed U$29: 9V-, 03lanfra-PADS:LITZENPAD
- removed U$30: 9VSW+, 03lanfra-PADS:LITZENPAD
- removed U$31: 9VSW-, 03lanfra-PADS:LITZENPAD
- added U$32, U$33, U$34, U$35, U$36: (no value), 03lanfra-PADS:MESSPAD
- moved R32 78.9 mm to (87.7, 53.3), turned to 0 degrees
- moved U$26 59.7 mm to (79.0, 50.2)
- moved JP4 58.5 mm to (78.8, 41.2), turned to 270 degrees
- moved U$24 57.4 mm to (79.0, 31.8)
- moved U6 56.1 mm to (89.1, 41.4), turned to 180 degrees
- moved C10 48.0 mm to (79.2, 55.8), turned to 180 degrees
- moved U$17 45.2 mm to (53.9, 18.5)
- moved R14 42.6 mm to (15.6, 95.6), turned to 180 degrees
- moved R29 38.8 mm to (57.5, 48.2), turned to 0 degrees
- moved U$15 38.4 mm to (53.9, 21.0)
- moved U$25 38.4 mm to (79.0, 47.7)
- moved JP1 37.9 mm to (57.5, 19.6), turned to 270 degrees
- moved R31 37.6 mm to (95.8, 6.56)
- moved U$23 37.3 mm to (79.1, 34.3), flipped to the bottom
- moved T1 36.2 mm to (15.5, 92.1)
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Connections:
- removed net N$15: U$28.P$1, U$30.P$1
- removed net N$20: R20.2, U3.2
- removed net N$21: R21.2, U3.3
- removed net N$22: R22.2, U3.4
- removed net N$35: R17.2, U5.2
- removed net N$36: R18.2, U5.3
- removed net N$37: R19.2, U5.4
- removed net N$42: R23.2, U4.2
- removed net N$43: R24.2, U4.3
- removed net N$44: R25.2, U4.4
- removed net N$5: LTZPDVCC.P$1, U$1.P$1
- removed net N$53: R26.2, U6.2
- removed net N$54: R27.2, U6.3
- removed net N$55: R28.2, U6.4
- removed net N$57: X1.5
- removed net N$58: X1.6
- removed net N$59: X1.7
- removed net N$60: X1.8
- new net +VCC: U$33.MSP, X1.6, X1.7
- net 3V3: no longer R17.1, R18.1, R19.1, R20.1, R21.1, R22.1, R23.1, R24.1, R25.1, R26.1, R27.1, R28.1
- net 9V: now also U$35.MSP; no longer U$31.P$1
- net GND: now also U$32.MSP, X1.8; no longer U$10.MSP, U$27.P$1, U$29.P$1
- net N$4: no longer U$4.MSP
- net N$46: now also U$36.MSP
- net N$6: now also LED1.C
- net N$8: no longer U$2.MSP
- net N$9: no longer LED1.C
- net VCC: now also U$34.MSP, X1.5; no longer LTZPDGND.P$1
Routing:
- net DIR3: track 109.2 -> 0.00 mm, vias 5 -> 0
- net STEP3: track 101.6 -> 0.00 mm, vias 5 -> 0
- net PIN1: track 86.1 -> 0.00 mm, vias 2 -> 0
- net GND: track 142.3 -> 60.4 mm, vias 16 -> 10
- net 3V3: track 111.6 -> 45.5 mm, vias 17 -> 12
- net DTR: track 75.5 -> 9.63 mm
- net N$34: track 38.6 -> 0.00 mm
- net N$28: track 39.4 -> 3.80 mm
- net N$17: track 40.0 -> 8.02 mm
- net N$52: track 36.0 -> 4.01 mm
- net N$54: track 31.0 -> 0.00 mm, vias 2 -> 0
- net N$29: track 34.3 -> 3.80 mm
- net N$41: track 30.3 -> 0.00 mm, vias 1 -> 0
- net N$32: track 29.1 -> 0.00 mm
- net N$27: track 32.5 -> 3.80 mm, vias 1 -> 0
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
Commit message: Tried with PID loop
Routing:
- net PIN1: track 0.00 -> 74.6 mm, vias 0 -> 6
- net DTR: track 9.63 -> 82.7 mm, vias 0 -> 4
- net VCC: track 138.6 -> 180.5 mm, vias 1 -> 2
- net N$39: track 0.00 -> 30.7 mm
- net N$28: track 3.80 -> 15.9 mm
- net N$26: track 3.80 -> 15.2 mm
- net +VCC: track 0.00 -> 8.62 mm
- net N$29: track 3.80 -> 6.93 mm
- net N$27: track 3.80 -> 6.78 mm
